File: KiCad/Arduino.kicad_sch (KiCad schematic)
At the start: 17 parts, among them SW1 SW_Push, SW2 SW_Push

Commit message: updated milestone and kicad
Parts:
- removed R1: 1k, symbol Device:R
- removed R2: 2k, symbol Device:R
Connections:
- net ECHO: now also A1.11 (D8)
Other:
- note added: "logic level converters"
- moved on the sheet: A1, R3, R4, R5, R6, R7, SW1, SW2, U1, U2

Commit message: added certificates
Parts:
- added R12: 10k, symbol Device:R
- added R13: 20k, symbol Device:R
Connections:
- net ECHO: now also R12.1; no longer A1.11 (D8)
- net GND: now also R13.2
- new net: A1.11 (D8), R12.2, R13.1
Changed lines of the file:
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@@
   (junction (at 146.05 76.2) (diameter 0) (color 0 0 0 0)
+  )
+  (junction (at 66.04 75.565) (diameter 0) (color 0 0 0 0)
   )
   (no_connect (at 109.22 63.5))
@@
     (stroke (width 0) (type default))
   )
+  (wire (pts (xy 66.04 74.295) (xy 66.04 75.565))
+    (stroke (width 0) (type default))
+  )
   (wire (pts (xy 73.66 40.64) (xy 73.66 50.8))
     (stroke (width 0) (type default))
   )
+  (wire (pts (xy 73.66 75.565) (xy 73.66 63.5))
+    (stroke (width 0) (type default))
+  )
   (wire (pts (xy 96.52 86.36) (xy 96.52 88.9))
     (stroke (width 0) (type default))
@@
     (stroke (width 0) (type default))
   )
+  (wire (pts (xy 73.66 63.5) (xy 83.82 63.5))
+    (stroke (width 0) (type default))
+  )
   (wire (pts (xy 133.35 66.04) (xy 135.89 66.04))
     (stroke (width 0) (type default))
@@
     (stroke (width 0) (type default))
   )
+  (wire (pts (xy 66.04 75.565) (xy 66.04 77.47))
+    (stroke (width 0) (type default))
+  )
   (wire (pts (xy 60.96 58.42) (xy 83.82 58.42))
     (stroke (width 0) (type default))
@@
   )
   (wire (pts (xy 109.22 68.58) (xy 119.38 68.58))
+    (stroke (width 0) (type default))
+  )
+  (wire (pts (xy 66.04 75.565) (xy 73.66 75.565))
     (stroke (width 0) (type default))
   )
@@
     (effects (font (size 1.27 1.27)) (justify left bottom))
   )
+  (hierarchical_label "GND" (shape input) (at 66.04 85.09 270) (fields_autoplaced)
+    (effects (font (size 1.27 1.27)) (justify right))
+  )
   (hierarchical_label "5V" (shape input) (at 45.72 53.34 180) (fields_autoplaced)
     (effects (font (size 1.27 1.27)) (justify right))
@@
     (effects (font (size 1.27 1.27)) (justify right))
   )
-  (hierarchical_label "ECHO" (shape input) (at 83.82 63.5 180) (fields_autoplaced)
+  (hierarchical_label "ECHO" (shape input) (at 66.04 66.675 180) (fields_autoplaced)
     (effects (font (size 1.27 1.27)) (justify right))
   )
@@
     )
   )
+  (symbol (lib_id "Device:R") (at 66.04 70.485 0) (unit 1)
+    (in_bom yes) (on_board yes) (dnp no) (fields_autoplaced)
+    (property "Reference" "R12" (at 68.58 69.85 0)
+      (effects (font (size 1.27 1.27)) (justify left))
+    )
+    (property "Value" "10k" (at 68.58 72.39 0)
+      (effects (font (size 1.27 1.27)) (justify left))
+    )
+    (property "Footprint" "" (at 64.262 70.485 90)
+      (effects (font (size 1.27 1.27)) hide)
+    )
+    (property "Datasheet" "~" (at 66.04 70.485 0)
+      (effects (font (size 1.27 1.27)) hide)
+    )
+    (pin "1")
+    (pin "2")
+    (instances
+      (project "KiCad"
+        (path "/c844c981-873d-46aa-90d6-aac9bb94e4aa/1540c02b-6fc2-48b2-8faf-4073a8443eef"
+          (reference "R12") (unit 1)
+        )
+      )
+    )
+  )
   (symbol (lib_id "Device:R") (at 139.7 60.96 90) (unit 1)
     (in_bom yes) (on_board yes) (dnp no)
@@
         )
       )
+    )
+  )
+  (symbol (lib_id "Device:R") (at 66.04 81.28 0) (unit 1)
+    (in_bom yes) (on_board yes) (dnp no) (fields_autoplaced)
+    (property "Reference" "R13" (at 68.58 80.645 0)
+      (effects (font (size 1.27 1.27)) (justify left))
+    )
+    (property "Value" "20k" (at 68.58 83.185 0)
+      (effects (font (size 1.27 1.27)) (justify left))
+    )
+    (property "Footprint" "" (at 64.262 81.28 90)
+      (effects (font (size 1.27 1.27)) hide)
+    )
+    (property "Datasheet" "~" (at 66.04 81.28 0)
+      (effects (font (size 1.27 1.27)) hide)
+    )
+    (pin "1")
+    (pin "2")
+    (instances
+      (project "KiCad"
+        (path "/c844c981-873d-46aa-90d6-aac9bb94e4aa/1540c02b-6fc2-48b2-8faf-4073a8443eef"
+          (reference "R13") (unit 1)
+        )
+      )

Commit message: made folder for milestone 3
Parts:
- added R14: 10k, symbol Device:R
- added R15: 20k, symbol Device:R
Connections:
- net ECHO: now also U1. (LV4); no longer R12.1
- net GND: now also R15.2
- net SIGL: now also R14.1; no longer U1. (LV4)
- net SIGR: now also R12.1; no longer U1. (LV4)
- net TRIG: now also U1. (LV4); no longer A1.12 (D9)
- new net: A1.12 (D9), R14.2, R15.1
Other:
- moved on the sheet: R12, R13
Changed lines of the file:
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@@
   (junction (at 146.05 81.28) (diameter 0) (color 0 0 0 0)
   )
+  (junction (at 57.15 79.375) (diameter 0) (color 0 0 0 0)
+  )
   (junction (at 146.05 55.88) (diameter 0) (color 0 0 0 0)
   )
@@
   (junction (at 146.05 60.96) (diameter 0) (color 0 0 0 0)
   )
+  (junction (at 66.04 77.47) (diameter 0) (color 0 0 0 0)
+  )
   (junction (at 146.05 76.2) (diameter 0) (color 0 0 0 0)
-  )
-  (junction (at 66.04 75.565) (diameter 0) (color 0 0 0 0)
   )
   (no_connect (at 109.22 63.5))
@@
     (stroke (width 0) (type default))
   )
-  (wire (pts (xy 66.04 74.295) (xy 66.04 75.565))
+  (wire (pts (xy 66.04 76.2) (xy 66.04 77.47))
     (stroke (width 0) (type default))
   )
@@
     (stroke (width 0) (type default))
   )
-  (wire (pts (xy 73.66 75.565) (xy 73.66 63.5))
-    (stroke (width 0) (type default))
-  )
   (wire (pts (xy 96.52 86.36) (xy 96.52 88.9))
     (stroke (width 0) (type default))
@@
     (stroke (width 0) (type default))
   )
+  (wire (pts (xy 57.15 79.375) (xy 75.565 79.375))
+    (stroke (width 0) (type default))
+  )
   (wire (pts (xy 133.35 66.04) (xy 135.89 66.04))
     (stroke (width 0) (type default))
@@
     (stroke (width 0) (type default))
   )
-  (wire (pts (xy 66.04 75.565) (xy 66.04 77.47))
+  (wire (pts (xy 57.15 79.375) (xy 57.15 81.28))
+    (stroke (width 0) (type default))
+  )
+  (wire (pts (xy 73.66 63.5) (xy 73.66 77.47))
     (stroke (width 0) (type default))
   )
@@
     (stroke (width 0) (type default))
   )
+  (wire (pts (xy 66.04 77.47) (xy 66.04 81.28))
+    (stroke (width 0) (type default))
+  )
   (wire (pts (xy 116.84 76.2) (xy 116.84 81.28))
     (stroke (width 0) (type default))
@@
     (stroke (width 0) (type default))
   )
-  (wire (pts (xy 66.04 75.565) (xy 73.66 75.565))
+  (wire (pts (xy 66.04 77.47) (xy 73.66 77.47))
     (stroke (width 0) (type default))
   )
@@
     (stroke (width 0) (type default))
   )
+  (wire (pts (xy 75.565 66.04) (xy 83.82 66.04))
+    (stroke (width 0) (type default))
+  )
   (wire (pts (xy 78.74 45.72) (xy 83.82 45.72))
     (stroke (width 0) (type default))
@@
     (stroke (width 0) (type default))
   )
+  (wire (pts (xy 75.565 66.04) (xy 75.565 79.375))
+    (stroke (width 0) (type default))
+  )
   (wire (pts (xy 96.52 86.36) (xy 99.06 86.36))
     (stroke (width 0) (type default))
@@
   )
   (wire (pts (xy 146.05 60.96) (xy 146.05 55.88))
+    (stroke (width 0) (type default))
+  )
+  (wire (pts (xy 57.15 76.2) (xy 57.15 79.375))
     (stroke (width 0) (type default))
   )
@@
     (effects (font (size 1.27 1.27)) (justify left bottom))
   )
-  (hierarchical_label "GND" (shape input) (at 66.04 85.09 270) (fields_autoplaced)
+  (hierarchical_label "GND" (shape input) (at 66.04 88.9 270) (fields_autoplaced)
     (effects (font (size 1.27 1.27)) (justify right))
   )
@@
     (effects (font (size 1.27 1.27)) (justify right))
   )
-  (hierarchical_label "ECHO" (shape input) (at 66.04 66.675 180) (fields_autoplaced)
+  (hierarchical_label "ECHO" (shape input) (at 45.72 27.94 180) (fields_autoplaced)
     (effects (font (size 1.27 1.27)) (justify right))
   )
@@
     (effects (font (size 1.27 1.27)) (justify right))
   )
-  (hierarchical_label "SIGL" (shape input) (at 45.72 27.94 180) (fields_autoplaced)
+  (hierarchical_label "SIGL" (shape input) (at 57.15 68.58 180) (fields_autoplaced)
     (effects (font (size 1.27 1.27)) (justify right))
   )
@@
     (effects (font (size 1.27 1.27)) (justify right))
   )
+  (hierarchical_label "GND" (shape input) (at 57.15 88.9 270) (fields_autoplaced)
+    (effects (font (size 1.27 1.27)) (justify right))
+  )
   (hierarchical_label "IN3" (shape output) (at 45.72 58.42 180) (fields_autoplaced)
     (effects (font (size 1.27 1.27)) (justify right))
   )
-  (hierarchical_label "SIGR" (shape input) (at 45.72 30.48 180) (fields_autoplaced)
+  (hierarchical_label "SIGR" (shape input) (at 66.04 68.58 180) (fields_autoplaced)
     (effects (font (size 1.27 1.27)) (justify right))
   )
@@
     (effects (font (size 1.27 1.27)) (justify left))
   )
-  (hierarchical_label "TRIG" (shape output) (at 83.82 66.04 180) (fields_autoplaced)
-    (effects (font (size 1.27 1.27)) (justify right))
+  (hierarchical_label "TRIG" (shape output) (at 45.72 30.48 180) (fields_autoplaced)
+    (effects (font (size 1.27 1.27)) (justify right))
+  )
+  (symbol (lib_id "Device:R") (at 57.15 85.09 0) (unit 1)
+    (in_bom yes) (on_board yes) (dnp no) (fields_autoplaced)
+    (property "Reference" "R15" (at 59.69 84.455 0)
+      (effects (font (size 1.27 1.27)) (justify left))
+    )
+    (property "Value" "20k" (at 59.69 86.995 0)
+      (effects (font (size 1.27 1.27)) (justify left))
+    )
+    (property "Footprint" "" (at 55.372 85.09 90)
+      (effects (font (size 1.27 1.27)) hide)
+    )
+    (property "Datasheet" "~" (at 57.15 85.09 0)
+      (effects (font (size 1.27 1.27)) hide)
+    )
+    (pin "1")
+    (pin "2")
+    (instances
+      (project "KiCad"
+        (path "/c844c981-873d-46aa-90d6-aac9bb94e4aa/1540c02b-6fc2-48b2-8faf-4073a8443eef"
+          (reference "R15") (unit 1)
+        )
+      )
+    )
   )
   (symbol (lib_id "Device:LED") (at 129.54 66.04 180) (unit 1)
@@
         (path "/c844c981-873d-46aa-90d6-aac9bb94e4aa/1540c02b-6fc2-48b2-8faf-4073a8443eef"
           (reference "D2") (unit 1)
+        )
+      )
+    )
+  )
+  (symbol (lib_id "Device:R") (at 57.15 72.39 0) (unit 1)
+    (in_bom yes) (on_board yes) (dnp no) (fields_autoplaced)
+    (property "Reference" "R14" (at 59.69 71.755 0)
+      (effects (font (size 1.27 1.27)) (justify left))
+    )
+    (property "Value" "10k" (at 59.69 74.295 0)
+      (effects (font (size 1.27 1.27)) (justify left))
+    )
+    (property "Footprint" "" (at 55.372 72.39 90)
+      (effects (font (size 1.27 1.27)) hide)
+    )
+    (property "Datasheet" "~" (at 57.15 72.39 0)
+      (effects (font (size 1.27 1.27)) hide)
+    )
+    (pin "1")
+    (pin "2")
+    (instances
+      (project "KiCad"
+        (path "/c844c981-873d-46aa-90d6-aac9bb94e4aa/1540c02b-6fc2-48b2-8faf-4073a8443eef"
+          (reference "R14") (unit 1)
         )
       )
@@
     )
   )
-  (symbol (lib_id "Device:R") (at 66.04 70.485 0) (unit 1)
+  (symbol (lib_id "Device:R") (at 66.04 72.39 0) (unit 1)
     (in_bom yes) (on_board yes) (dnp no) (fields_autoplaced)
-    (property "Reference" "R12" (at 68.58 69.85 0)
-      (effects (font (size 1.27 1.27)) (justify left))
-    )
-    (property "Value" "10k" (at 68.58 72.39 0)
-      (effects (font (size 1.27 1.27)) (justify left))
-    )
-    (property "Footprint" "" (at 64.262 70.485 90)
-      (effects (font (size 1.27 1.27)) hide)
-    )
-    (property "Datasheet" "~" (at 66.04 70.485 0)
+    (property "Reference" "R12" (at 68.58 71.755 0)
+      (effects (font (size 1.27 1.27)) (justify left))
+    )
+    (property "Value" "10k" (at 68.58 74.295 0)
+      (effects (font (size 1.27 1.27)) (justify left))
+    )
+    (property "Footprint" "" (at 64.262 72.39 90)
+      (effects (font (size 1.27 1.27)) hide)
+    )
+    (property "Datasheet" "~" (at 66.04 72.39 0)
       (effects (font (size 1.27 1.27)) hide)
     )
@@
     )
   )
-  (symbol (lib_id "Device:R") (at 66.04 81.28 0) (unit 1)
+  (symbol (lib_id "Device:R") (at 66.04 85.09 0) (unit 1)
     (in_bom yes) (on_board yes) (dnp no) (fields_autoplaced)
-    (property "Reference" "R13" (at 68.58 80.645 0)
-      (effects (font (size 1.27 1.27)) (justify left))
-    )
-    (property "Value" "20k" (at 68.58 83.185 0)
-      (effects (font (size 1.27 1.27)) (justify left))
-    )
-    (property "Footprint" "" (at 64.262 81.28 90)
-      (effects (font (size 1.27 1.27)) hide)
-    )
-    (property "Datasheet" "~" (at 66.04 81.28 0)
-      (effects (font (size 1.27 1.27)) hide)
-    )
+    (property "Reference" "R13" (at 68.58 84.455 0)
+      (effects (font (size 1.27 1.27)) (justify left))
+    )
+    (property "Value" "20k" (at 68.58 86.995 0)
+      (effects (font (size 1.27 1.27)) (justify left))
+    )
+    (property "Footprint" "" (at 64.262 85.09 90)
+      (effects (font (size 1.27 1.27)) hide)
+    )
+    (property "Datasheet" "~" (at 66.04 85.09 0)
+      (effects (font (size 1.27 1.27)) hide)
+    )

Commit message: ki cad changes
Parts:
- removed D1: LED_BLUE, symbol Device:LED
- removed D2: LED_WHITE, symbol Device:LED
- removed D5: LED_RED, symbol Device:LED
- removed R3, R4, R7: 1.2k, symbol Device:R
- removed SW2: SW_Push, symbol Switch:SW_Push
- added R16: 10k, symbol Device:R
- D4: value LED_ORANGE -> LED_YELLOW
Connections:
- net 3V3: now also A1.18 (AREF), R16.1
- net LINE1: now also A1.21 (A2); no longer A1.13 (D10)
- net LINE2: now also A1.22 (A3); no longer A1.14 (D11)
- net LINE3: now also A1.25 (A6); no longer A1.15 (D12)
- net LINE4: now also A1.26 (A7); no longer A1.16 (D13)
- net at A1.19 (A0), SW1.1: now also R16.2
- net at D3.2 (A): now also A1.16 (D13); no longer A1.24 (A5)
- net at A1.1 (D1/TX): no longer U1. (LV4)
- net at A1.2 (D0/RX): no longer U1. (LV4)
- net at R12.2, R13.1: now also A1.13 (D10); no longer A1.11 (D8)
- net at D4.2 (A): now also A1.15 (D12); no longer A1.25 (A6)
- new net: A1.11 (D8), U1. (LV4)
- new net: A1.14 (D11), U1. (LV4)
- no-connect marks 5 -> 6

Commit message: kicad
Connections:
- net 5V: no longer A1.30 (VIN)
- new net 7.5V: A1.30 (VIN)
Changed lines of the file:
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@@
     (stroke (width 0) (type default))
   )
-  (wire (pts (xy 99.06 30.48) (xy 99.06 31.75))
+  (wire (pts (xy 99.06 29.21) (xy 99.06 31.75))
     (stroke (width 0) (type default))
   )
@@
     (effects (font (size 1.27 1.27)) (justify right))
   )
-  (hierarchical_label "3V3" (shape output) (at 99.06 30.48 90) (fields_autoplaced)
+  (hierarchical_label "3V3" (shape output) (at 99.06 29.21 90) (fields_autoplaced)
     (effects (font (size 1.27 1.27)) (justify left))
   )
@@
   (hierarchical_label "ECHO" (shape input) (at 45.72 27.94 180) (fields_autoplaced)
     (effects (font (size 1.27 1.27)) (justify right))
-  )
-  (hierarchical_label "5V" (shape input) (at 93.98 30.48 90) (fields_autoplaced)
-    (effects (font (size 1.27 1.27)) (justify left))
   )
   (hierarchical_label "IN2" (shape output) (at 45.72 50.8 180) (fields_autoplaced)
@@
     (effects (font (size 1.27 1.27)) (justify left))
   )
+  (hierarchical_label "7.5V" (shape output) (at 93.98 30.48 90) (fields_autoplaced)
+    (effects (font (size 1.27 1.27)) (justify left))
+  )
