File: KiCad/H-Bridge.kicad_sch (KiCad schematic)
At the start: 0 parts

Commit message: kicad
Changed lines of the file:
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@@
     (comment 1 "Author: Cameron Clark")
   )
-  (hierarchical_label "ENB" (shape input) (at 218.44 116.84 270) (fields_autoplaced)
+  (rectangle (start 200.66 134.62) (end 233.68 162.56)
+    (stroke (width 0) (type default))
+    (fill (type none))
+  )
+  (hierarchical_label "ENB" (shape input) (at 231.14 134.62 270) (fields_autoplaced)
     (effects (font (size 1.27 1.27)) (justify right))
   )
-  (hierarchical_label "GND" (shape input) (at 203.2 144.78 90) (fields_autoplaced)
+  (hierarchical_label "GND" (shape input) (at 215.9 162.56 90) (fields_autoplaced)
     (effects (font (size 1.27 1.27)) (justify left))
   )
-  (hierarchical_label "OUT4" (shape output) (at 220.98 129.54 180) (fields_autoplaced)
+  (hierarchical_label "OUT4" (shape output) (at 233.68 147.32 180) (fields_autoplaced)
     (effects (font (size 1.27 1.27)) (justify right))
   )
-  (hierarchical_label "ENA" (shape input) (at 193.04 116.84 270) (fields_autoplaced)
+  (hierarchical_label "ENA" (shape input) (at 205.74 134.62 270) (fields_autoplaced)
     (effects (font (size 1.27 1.27)) (justify right))
   )
-  (hierarchical_label "IN1" (shape input) (at 198.12 116.84 270) (fields_autoplaced)
+  (hierarchical_label "IN1" (shape input) (at 210.82 134.62 270) (fields_autoplaced)
     (effects (font (size 1.27 1.27)) (justify right))
   )
-  (hierarchical_label "12V" (shape input) (at 198.12 144.78 90) (fields_autoplaced)
+  (hierarchical_label "12V" (shape input) (at 210.82 162.56 90) (fields_autoplaced)
     (effects (font (size 1.27 1.27)) (justify left))
   )
-  (hierarchical_label "OUT1" (shape output) (at 187.96 129.54 0) (fields_autoplaced)
+  (hierarchical_label "OUT1" (shape output) (at 200.66 147.32 0) (fields_autoplaced)
     (effects (font (size 1.27 1.27)) (justify left))
   )
-  (hierarchical_label "IN4" (shape input) (at 213.36 116.84 270) (fields_autoplaced)
+  (hierarchical_label "IN4" (shape input) (at 226.06 134.62 270) (fields_autoplaced)
     (effects (font (size 1.27 1.27)) (justify right))
   )
-  (hierarchical_label "OUT3" (shape output) (at 220.98 134.62 180) (fields_autoplaced)
+  (hierarchical_label "OUT3" (shape output) (at 233.68 152.4 180) (fields_autoplaced)
     (effects (font (size 1.27 1.27)) (justify right))
   )
-  (hierarchical_label "IN3" (shape input) (at 208.28 116.84 270) (fields_autoplaced)
+  (hierarchical_label "IN3" (shape input) (at 220.98 134.62 270) (fields_autoplaced)
     (effects (font (size 1.27 1.27)) (justify right))
   )
-  (hierarchical_label "OUT2" (shape output) (at 187.96 134.62 0) (fields_autoplaced)
+  (hierarchical_label "OUT2" (shape output) (at 200.66 152.4 0) (fields_autoplaced)
     (effects (font (size 1.27 1.27)) (justify left))
   )
-  (hierarchical_label "IN2" (shape input) (at 203.2 116.84 270) (fields_autoplaced)
+  (hierarchical_label "IN2" (shape input) (at 215.9 134.62 270) (fields_autoplaced)
     (effects (font (size 1.27 1.27)) (justify right))
   )
-  (hierarchical_label "5V" (shape input) (at 208.28 144.78 90) (fields_autoplaced)
+  (hierarchical_label "5V" (shape input) (at 220.98 162.56 90) (fields_autoplaced)
     (effects (font (size 1.27 1.27)) (justify left))
   )
