File: KiCad/KiCad.kicad_sch (KiCad schematic)
At the start: 0 parts

Commit message: kicad
Other:
- sheet Arduino ports: added 7.5V; removed 5V
- sheet Power ports: added 7.5V arduino, 7.5V switch; removed none
Changed lines of the file:
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@@
     (comment 1 "Author: Cameron Clark")
   )
-  (junction (at 15.24 48.26) (diameter 0) (color 0 0 0 0)
-  )
   (junction (at 86.36 25.4) (diameter 0) (color 0 0 0 0)
   )
@@
     (stroke (width 0) (type default))
   )
+  (wire (pts (xy 53.34 93.98) (xy 53.34 105.41))
+    (stroke (width 0) (type default))
+  )
   (wire (pts (xy 45.72 27.94) (xy 45.72 43.18))
     (stroke (width 0) (type default))
@@
     (stroke (width 0) (type default))
   )
+  (wire (pts (xy 13.97 100.33) (xy 13.97 48.26))
+    (stroke (width 0) (type default))
+  )
   (wire (pts (xy 17.78 66.04) (xy 17.78 96.52))
     (stroke (width 0) (type default))
@@
     (stroke (width 0) (type default))
   )
+  (wire (pts (xy 66.04 115.57) (xy 66.04 116.84))
+    (stroke (width 0) (type default))
+  )
   (wire (pts (xy 63.5 93.98) (xy 63.5 99.06))
     (stroke (width 0) (type default))
@@
     (stroke (width 0) (type default))
   )
+  (wire (pts (xy 46.99 100.33) (xy 13.97 100.33))
+    (stroke (width 0) (type default))
+  )
   (wire (pts (xy 27.94 86.36) (xy 35.56 86.36))
     (stroke (width 0) (type default))
@@
     (stroke (width 0) (type default))
   )
-  (wire (pts (xy 35.56 48.26) (xy 15.24 48.26))
-    (stroke (width 0) (type default))
-  )
   (wire (pts (xy 101.6 96.52) (xy 101.6 66.04))
     (stroke (width 0) (type default))
@@
     (stroke (width 0) (type default))
   )
+  (wire (pts (xy 58.42 96.52) (xy 101.6 96.52))
+    (stroke (width 0) (type default))
+  )
   (wire (pts (xy 60.96 40.64) (xy 60.96 43.18))
     (stroke (width 0) (type default))
@@
     (stroke (width 0) (type default))
   )
-  (wire (pts (xy 15.24 48.26) (xy 15.24 63.5))
-    (stroke (width 0) (type default))
-  )
-  (wire (pts (xy 58.42 96.52) (xy 101.6 96.52))
+  (wire (pts (xy 46.99 105.41) (xy 46.99 100.33))
+    (stroke (width 0) (type default))
+  )
+  (wire (pts (xy 15.24 35.56) (xy 15.24 63.5))
     (stroke (width 0) (type default))
   )
@@
     (stroke (width 0) (type default))
   )
-  (wire (pts (xy 58.42 96.52) (xy 58.42 101.6))
+  (wire (pts (xy 58.42 96.52) (xy 58.42 105.41))
     (stroke (width 0) (type default))
   )
@@
     (stroke (width 0) (type default))
   )
-  (wire (pts (xy 15.24 35.56) (xy 15.24 48.26))
-    (stroke (width 0) (type default))
-  )
   (wire (pts (xy 15.24 63.5) (xy 20.32 63.5))
     (stroke (width 0) (type default))
@@
     (stroke (width 0) (type default))
   )
+  (wire (pts (xy 13.97 48.26) (xy 35.56 48.26))
+    (stroke (width 0) (type default))
+  )
   (wire (pts (xy 58.42 78.74) (xy 58.42 81.28))
     (stroke (width 0) (type default))
@@
     (stroke (width 0) (type default))
   )
-  (wire (pts (xy 63.5 99.06) (xy 63.5 101.6))
+  (wire (pts (xy 63.5 99.06) (xy 63.5 105.41))
     (stroke (width 0) (type default))
   )
@@
       (effects (font (size 1.27 1.27)) (justify left))
     )
-    (pin "5V" input (at 35.56 48.26 180)
-      (effects (font (size 1.27 1.27)) (justify left))
-    )
     (pin "3V3" output (at 35.56 45.72 180)
+      (effects (font (size 1.27 1.27)) (justify left))
+    )
+    (pin "7.5V" output (at 35.56 48.26 180)
       (effects (font (size 1.27 1.27)) (justify left))
     )
@@
     )
   )
-  (sheet (at 35.56 101.6) (size 48.26 10.16)
+  (sheet (at 35.56 105.41) (size 48.26 15.24)
     (stroke (width 0.1524) (type solid))
     (fill (color 0 0 0 0.0000))
-    (property "Sheetname" "Power" (at 35.56 101.6 0)
+    (property "Sheetname" "Power" (at 35.56 105.41 0)
       (effects (font (size 1.27 1.27)) (justify left bottom))
     )
-    (property "Sheetfile" "Power.kicad_sch" (at 84.4046 111.76 90)
+    (property "Sheetfile" "Power.kicad_sch" (at 84.4046 115.57 90)
       (effects (font (size 1.27 1.27)) (justify left top) hide)
     )
-    (pin "5V" output (at 63.5 101.6 90)
-      (effects (font (size 1.27 1.27)) (justify right))
-    )
-    (pin "GND" output (at 58.42 101.6 90)
-      (effects (font (size 1.27 1.27)) (justify right))
-    )
+    (pin "5V" output (at 63.5 105.41 90)
+      (effects (font (size 1.27 1.27)) (justify right))
+    )
+    (pin "GND" output (at 58.42 105.41 90)
+      (effects (font (size 1.27 1.27)) (justify right))
+    )
+    (pin "7.5V arduino" output (at 46.99 105.41 90)
+      (effects (font (size 1.27 1.27)) (justify right))
+    )
+    (pin "7.5V switch" output (at 53.34 105.41 90)
+      (effects (font (size 1.27 1.27)) (justify right))
+    )
