File: KiCad/LineSensor.kicad_sch (KiCad schematic)
At the start: 0 parts

Commit message: kicad
Changed lines of the file:
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@@
     (comment 1 "Author: Cameron Clark")
   )
-  (rectangle (start 156.21 125.73) (end 173.99 138.43)
+  (rectangle (start 185.42 151.13) (end 203.2 163.83)
     (stroke (width 0) (type default))
     (fill (type none))
   )
-  (rectangle (start 175.26 125.73) (end 193.04 138.43)
+  (rectangle (start 204.47 151.13) (end 222.25 163.83)
     (stroke (width 0) (type default))
     (fill (type none))
   )
-  (rectangle (start 213.36 125.73) (end 231.14 138.43)
+  (rectangle (start 242.57 151.13) (end 260.35 163.83)
     (stroke (width 0) (type default))
     (fill (type none))
   )
-  (rectangle (start 194.31 125.73) (end 212.09 138.43)
+  (rectangle (start 223.52 151.13) (end 241.3 163.83)
     (stroke (width 0) (type default))
     (fill (type none))
   )
-  (hierarchical_label "SIG_2" (shape output) (at 184.15 125.73 270) (fields_autoplaced)
+  (hierarchical_label "SIG_2" (shape output) (at 213.36 151.13 270) (fields_autoplaced)
     (effects (font (size 1.27 1.27)) (justify right))
   )
-  (hierarchical_label "3V3_2" (shape input) (at 180.34 125.73 270) (fields_autoplaced)
+  (hierarchical_label "3V3_2" (shape input) (at 209.55 151.13 270) (fields_autoplaced)
     (effects (font (size 1.27 1.27)) (justify right))
   )
-  (hierarchical_label "GND_1" (shape input) (at 168.91 125.73 270) (fields_autoplaced)
+  (hierarchical_label "GND_1" (shape input) (at 198.12 151.13 270) (fields_autoplaced)
     (effects (font (size 1.27 1.27)) (justify right))
   )
-  (hierarchical_label "3V3_4" (shape input) (at 218.44 125.73 270) (fields_autoplaced)
+  (hierarchical_label "3V3_4" (shape input) (at 247.65 151.13 270) (fields_autoplaced)
     (effects (font (size 1.27 1.27)) (justify right))
   )
-  (hierarchical_label "SIG_4" (shape output) (at 222.25 125.73 270) (fields_autoplaced)
+  (hierarchical_label "SIG_4" (shape output) (at 251.46 151.13 270) (fields_autoplaced)
     (effects (font (size 1.27 1.27)) (justify right))
   )
-  (hierarchical_label "SIG_3" (shape output) (at 203.2 125.73 270) (fields_autoplaced)
+  (hierarchical_label "SIG_3" (shape output) (at 232.41 151.13 270) (fields_autoplaced)
     (effects (font (size 1.27 1.27)) (justify right))
   )
-  (hierarchical_label "3V3_1" (shape input) (at 161.29 125.73 270) (fields_autoplaced)
+  (hierarchical_label "3V3_1" (shape input) (at 190.5 151.13 270) (fields_autoplaced)
     (effects (font (size 1.27 1.27)) (justify right))
   )
-  (hierarchical_label "GND_4" (shape input) (at 226.06 125.73 270) (fields_autoplaced)
+  (hierarchical_label "GND_4" (shape input) (at 255.27 151.13 270) (fields_autoplaced)
     (effects (font (size 1.27 1.27)) (justify right))
   )
-  (hierarchical_label "GND_3" (shape input) (at 207.01 125.73 270) (fields_autoplaced)
+  (hierarchical_label "GND_3" (shape input) (at 236.22 151.13 270) (fields_autoplaced)
     (effects (font (size 1.27 1.27)) (justify right))
   )
-  (hierarchical_label "GND_2" (shape input) (at 187.96 125.73 270) (fields_autoplaced)
+  (hierarchical_label "GND_2" (shape input) (at 217.17 151.13 270) (fields_autoplaced)
     (effects (font (size 1.27 1.27)) (justify right))
   )
-  (hierarchical_label "3V3_3" (shape input) (at 199.39 125.73 270) (fields_autoplaced)
+  (hierarchical_label "3V3_3" (shape input) (at 228.6 151.13 270) (fields_autoplaced)
     (effects (font (size 1.27 1.27)) (justify right))
   )
-  (hierarchical_label "SIG_1" (shape output) (at 165.1 125.73 270) (fields_autoplaced)
+  (hierarchical_label "SIG_1" (shape output) (at 194.31 151.13 270) (fields_autoplaced)
     (effects (font (size 1.27 1.27)) (justify right))
   )
