File: KiCad/MotorL.kicad_sch (KiCad schematic)
At the start: 0 parts

Commit message: kicad
Other:
- note added: "Encoder"
- note added: "motor"
Changed lines of the file:
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@@
     (comment 1 "Author: Cameron Clark")
+  )
+  (rectangle (start 179.07 146.05) (end 191.77 161.29)
+    (stroke (width 0) (type default))
+    (fill (type none))
+  )
+  (rectangle (start 209.55 144.78) (end 222.25 162.56)
+    (stroke (width 0) (type default))
+    (fill (type none))
+  )
+  (text "Encoder" (at 210.82 148.59 0)
+    (effects (font (size 1.27 1.27)) (justify left bottom))
+  )
+  (text "motor" (at 180.34 149.86 0)
+    (effects (font (size 1.27 1.27)) (justify left bottom))
   )
   (hierarchical_label "5VM" (shape input) (at 180.34 152.4 0) (fields_autoplaced)
