File: KiCad/MotorR.kicad_sch (KiCad schematic)
At the start: 0 parts

Commit message: kicad
Other:
- note added: "Encoder"
- note added: "motor"
Changed lines of the file:
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@@
     (comment 1 "Author: Cameron Clark")
+  )
+  (rectangle (start 208.28 146.05) (end 220.98 163.83)
+    (stroke (width 0) (type default))
+    (fill (type none))
+  )
+  (rectangle (start 177.8 147.32) (end 190.5 162.56)
+    (stroke (width 0) (type default))
+    (fill (type none))
+  )
+  (text "Encoder" (at 209.55 149.86 0)
+    (effects (font (size 1.27 1.27)) (justify left bottom))
+  )
+  (text "motor" (at 179.07 151.13 0)
+    (effects (font (size 1.27 1.27)) (justify left bottom))
   )
   (hierarchical_label "GNDM" (shape input) (at 179.705 158.115 0) (fields_autoplaced)
