File: KiCad/Ultrasonic.kicad_sch (KiCad schematic)
At the start: 0 parts

Commit message: kicad
Changed lines of the file:
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@@
     (comment 1 "Author: Cameron Clark")
   )
-  (hierarchical_label "5V" (shape input) (at 208.28 152.4 0) (fields_autoplaced)
-    (effects (font (size 1.27 1.27)) (justify left))
+  (rectangle (start 214.63 148.59) (end 246.38 156.21)
+    (stroke (width 0) (type default))
+    (fill (type none))
   )
-  (hierarchical_label "ECHO" (shape output) (at 215.9 152.4 0) (fields_autoplaced)
-    (effects (font (size 1.27 1.27)) (justify left))
+  (hierarchical_label "5V" (shape input) (at 218.44 148.59 270) (fields_autoplaced)
+    (effects (font (size 1.27 1.27)) (justify right))
   )
-  (hierarchical_label "GND" (shape input) (at 238.4595 152.2697 0) (fields_autoplaced)
-    (effects (font (size 1.27 1.27)) (justify left))
+  (hierarchical_label "ECHO" (shape output) (at 226.06 148.59 270) (fields_autoplaced)
+    (effects (font (size 1.27 1.27)) (justify right))
   )
-  (hierarchical_label "TRIG" (shape input) (at 227.33 152.4 0) (fields_autoplaced)
-    (effects (font (size 1.27 1.27)) (justify left))
+  (hierarchical_label "GND" (shape input) (at 240.03 148.59 270) (fields_autoplaced)
+    (effects (font (size 1.27 1.27)) (justify right))
+  )
+  (hierarchical_label "TRIG" (shape input) (at 233.68 148.59 270) (fields_autoplaced)
+    (effects (font (size 1.27 1.27)) (justify right))
   )
 )
